Commit message: [checked] modified UR3 urdf for real robot (the file name remain ur3e)

File: urdf/ur3e_robotiq/ur3e_urdf.xacro (robot description, xacro)
@@ -1,10 +1,10 @@
 <?xml version="1.1"?>
-<robot name="ur3e" xmlns:xacro="http://ros.org/wiki/xacro">
+<robot name="ur3" xmlns:xacro="http://ros.org/wiki/xacro">
   <xacro:include filename="$(find ur_description)/urdf/ur_macro.xacro" />
   <!-- ur_type -->
-  <xacro:arg name="ur_type" default="ur3e"/>
+  <xacro:arg name="ur_type" default="ur3"/>
   <!-- ros2_control related parameters -->
   <xacro:arg name="robot_ip" default="192.168.1.101" />
-  <xacro:arg name="generate_ros2_control_tag" default="false"/>
+  <xacro:arg name="generate_ros2_control_tag" default="true"/>
   <!-- parameters -->
   <xacro:arg name="tf_prefix" default=""/>
@@ -14,5 +14,5 @@
   <xacro:arg name="safety_k_position" default="20"/>
   <!-- Simulation parameters -->
-  <xacro:arg name="use_fake_hardware" default="true" />
+  <xacro:arg name="use_fake_hardware" default="false" />
   <xacro:arg name="fake_sensor_commands" default="false" />
   <xacro:arg name="sim_gazebo" default="false" />
@@ -20,6 +20,6 @@
   <xacro:arg name="simulation_controllers" default="" />
   <!-- initial position for simulations (Fake Hardware, Gazebo, Ignition) -->
-  <xacro:arg name="initial_positions_file" default="$(find cartesian_controller_simulation)/config/initial_positions.yaml"/>
-  <xacro:property name="initial_positions_file" default="$(arg initial_positions_file)"/>
+  <!-- <xacro:arg name="initial_positions_file" default="$(find cartesian_controller_simulation)/config/initial_positions.yaml"/> -->
+  <!-- <xacro:property name="initial_positions_file" default="$(arg initial_positions_file)"/> -->
   <link name="world" />
   <joint name="world_joint" type="fixed">
@@ -37,17 +37,20 @@
       safety_k_position="$(arg safety_k_position)"
       joint_limits_parameters_file="$(find ur_description)/config/$(arg ur_type)/joint_limits.yaml"
-      kinematics_parameters_file="$(find ur_description)/config/$(arg ur_type)/default_kinematics.yaml"
+      kinematics_parameters_file="$(find cartesian_controllers_universal_robots)/config/test_calibration.yaml"
       physical_parameters_file="$(find ur_description)/config/$(arg ur_type)/physical_parameters.yaml"
       visual_parameters_file="$(find ur_description)/config/$(arg ur_type)/visual_parameters.yaml"
+      script_filename="$(find ur_client_library)/resources/external_control.urscript"
+      input_recipe_filename="$(find ur_robot_driver)/resources/rtde_input_recipe.txt"
+      output_recipe_filename="$(find ur_robot_driver)/resources/rtde_output_recipe.txt"
       use_fake_hardware="$(arg use_fake_hardware)"
       fake_sensor_commands="$(arg fake_sensor_commands)"
       sim_gazebo="$(arg sim_gazebo)"
-      sim_ignition="$(arg sim_ignition)"
-      initial_positions="${xacro.load_yaml(initial_positions_file)}">
+      sim_ignition="$(arg sim_ignition)">
+      <!-- initial_positions="${xacro.load_yaml(initial_positions_file)}" -->
     <origin xyz="0 0.0 0.0" rpy="0 0 0" />
   </xacro:ur_robot>
   <xacro:include filename="$(find cartesian_controller_simulation)/urdf/joint.urdf.xacro"/>
   <!-- the parameter is modified for UR3e in mujoco -->
-  <ros2_control name="cartesian_controller_simulation" type="system">
+  <!-- <ros2_control name="cartesian_controller_simulation" type="system">
     <xacro:joint_interface name="shoulder_pan_joint" p="1000" d="100" />
     <xacro:joint_interface name="shoulder_lift_joint" p="1000" d="100" />
@@ -60,5 +63,5 @@
       <param name="mujoco_model">$(arg mujoco_model)</param>
     </hardware>
-  </ros2_control>
+  </ros2_control> -->
   <!-- <gazebo>
     <plugin filename="libgazebo_ros2_control.so" name="gazebo_ros2_control">
